File: hardware/power-supply-bricklet.kicad_pcb (KiCad board)
At the start: 2 copper layers, 40 x 25 mm, 38 parts, among them J101 green, P1 CON-SENSOR, P2 Debug, P3 Boot, U1 XMC1100, U101 MCP4551T-104E/MS, U102 TLV61046A, U3 DRILL, U4 DRILL, U5 DRILL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

Commit message: add fiducials, ordered version
Parts:
- added Fiducial_Mark: VAL**, kicad-libraries:Fiducial_Mark, F.Cu at (153.8, 101.6)
- added Fiducial_Mark: VAL**, kicad-libraries:Fiducial_Mark, F.Cu at (147.8, 79.6)
- added Fiducial_Mark: VAL**, kicad-libraries:Fiducial_Mark, F.Cu at (127.3, 82.0)
Changed lines of the file:
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@@
-(kicad_pcb (version 20171130) (host pcbnew 5.0.1-33cea8e~68~ubuntu18.04.1)
+(kicad_pcb (version 20171130) (host pcbnew 5.0.2-bee76a0~70~ubuntu18.04.1)
   (general
     (thickness 1.6002)
@@
     (tracks 359)
     (zones 0)
-    (modules 38)
+    (modules 41)
     (nets 28)
   )
@@
   )
   (setup
-    (last_trace_width 0.4)
+    (last_trace_width 0.2)
     (user_trace_width 0.2)
     (user_trace_width 0.25)
@@
     (pad_drill 0)
     (pad_to_mask_clearance 0)
-    (solder_mask_min_width 0.25)
     (aux_axis_origin 176.9 165.9)
     (grid_origin 176.9 165.9)
     (visible_elements FFFFFFBF)
     (pcbplotparams
-      (layerselection 0x010f0_80000001)
+      (layerselection 0x010fc_ffffffff)
       (usegerberextensions true)
-      (usegerberattributes false)
+      (usegerberattributes true)
       (usegerberadvancedattributes false)
       (creategerberjobfile false)
       (excludeedgelayer true)
       (linewidth 0.150000)
-      (plotframeref true)
+      (plotframeref false)
       (viasonmask false)
       (mode 1)
@@
       (plotinvisibletext false)
       (padsonsilk false)
-      (subtractmaskfromsilk false)
+      (subtractmaskfromsilk true)
       (outputformat 1)
       (mirror false)
       (drillshape 0)
       (scaleselection 1)
-      (outputdirectory "/tmp/prod/"))
+      (outputdirectory "pcb/"))
   )
   (net 0 "")
@@
       (xy -0.55372 -1.41224) (xy -0.55372 -1.67132)) (layer B.SilkS) (width 0.00254))
   )
+  (module kicad-libraries:Fiducial_Mark (layer Vorderseite)
+    (at 153.8 101.6)
+    (attr smd)
+    (fp_text reference Fiducial_Mark (at 0 0) (layer F.SilkS) hide
+      (effects (font (size 0.127 0.127) (thickness 0.03302)))
+    )
+    (fp_text value VAL** (at 0 -0.29972) (layer F.SilkS) hide
+      (effects (font (size 0.127 0.127) (thickness 0.03302)))
+    )
+    (fp_circle (center 0 0) (end 1.15062 0) (layer Dwgs.User) (width 0.01016))
+    (pad 1 smd circle (at 0 0) (size 1.00076 1.00076) (layers Vorderseite F.Paste F.Mask)
+      (clearance 0.65024))
+  )
+  (module kicad-libraries:Fiducial_Mark (layer Vorderseite)
+    (at 147.8 79.6)
+    (attr smd)
+    (fp_text reference Fiducial_Mark (at 0 0) (layer F.SilkS) hide
+      (effects (font (size 0.127 0.127) (thickness 0.03302)))
+    )
+    (fp_text value VAL** (at 0 -0.29972) (layer F.SilkS) hide
+      (effects (font (size 0.127 0.127) (thickness 0.03302)))
+    )
+    (fp_circle (center 0 0) (end 1.15062 0) (layer Dwgs.User) (width 0.01016))
+    (pad 1 smd circle (at 0 0) (size 1.00076 1.00076) (layers Vorderseite F.Paste F.Mask)
+      (clearance 0.65024))
+  )
+  (module kicad-libraries:Fiducial_Mark (layer Vorderseite)
+    (at 127.3 82)
+    (attr smd)
+    (fp_text reference Fiducial_Mark (at 0 0) (layer F.SilkS) hide
+      (effects (font (size 0.127 0.127) (thickness 0.03302)))
+    )
+    (fp_text value VAL** (at 0 -0.29972) (layer F.SilkS) hide
+      (effects (font (size 0.127 0.127) (thickness 0.03302)))
+    )
+    (fp_circle (center 0 0) (end 1.15062 0) (layer Dwgs.User) (width 0.01016))
+    (pad 1 smd circle (at 0 0) (size 1.00076 1.00076) (layers Vorderseite F.Paste F.Mask)
+      (clearance 0.65024))
+  )
   (gr_text Output (at 156.3 85.4) (layer F.SilkS)
     (effects (font (size 0.7 0.7) (thickness 0.15)))
@@
   (segment (start 147.1 100.2) (end 145.8 101.5) (width 0.25) (layer Rückseite) (net 2))
   (segment (start 147.1 100.2) (end 147.1 99.8) (width 0.25) (layer Rückseite) (net 2))
-  (segment (start 143.1 101.5) (end 151.2 101.5) (width 0.25) (layer Vorderseite) (net 2))
-  (segment (start 156.8 95.9) (end 157.95 95.9) (width 0.25) (layer Vorderseite) (net 2) (status 800000))
-  (segment (start 151.2 101.5) (end 156.8 95.9) (width 0.25) (layer Vorderseite) (net 2))
+  (segment (start 143.1 101.5) (end 151.1 101.5) (width 0.25) (layer Vorderseite) (net 2))
+  (segment (start 156.7 95.9) (end 157.95 95.9) (width 0.25) (layer Vorderseite) (net 2) (status 800000))
+  (segment (start 151.1 101.5) (end 156.7 95.9) (width 0.25) (layer Vorderseite) (net 2))
   (segment (start 132.3 102) (end 127.5 102) (width 0.55) (layer Rückseite) (net 2))
   (segment (start 129.85 90.05) (end 129.1 90.05) (width 0.55) (layer Vorderseite) (net 2) (status 800000))
@@
   (segment (start 130.55 93.65) (end 130.55 96.475) (width 0.25) (layer Vorderseite) (net 13) (status 800000))
   (segment (start 129.3507 92.4507) (end 130.55 93.65) (width 0.25) (layer Vorderseite) (net 13))
-  (segment (start 137.3509 102.09888) (end 151.50112 102.09888) (width 0.25) (layer Vorderseite) (net 14) (status 400000))
+  (segment (start 137.3509 102.09888) (end 151.40112 102.09888) (width 0.25) (layer Vorderseite) (net 14) (status 400000))
   (segment (start 159.4 95.9) (end 159.45 95.9) (width 0.25) (layer Vorderseite) (net 14) (status C00000))
   (segment (start 159.4 96.5) (end 159.4 95.9) (width 0.25) (layer Vorderseite) (net 14) (status 800000))
   (segment (start 158.9 97) (end 159.4 96.5) (width 0.25) (layer Vorderseite) (net 14))
-  (segment (start 156.6 97) (end 158.9 97) (width 0.25) (layer Vorderseite) (net 14))
-  (segment (start 151.50112 102.09888) (end 156.6 97) (width 0.25) (layer Vorderseite) (net 14))
+  (segment (start 156.5 97) (end 158.9 97) (width 0.25) (layer Vorderseite) (net 14))
+  (segment (start 151.40112 102.09888) (end 156.5 97) (width 0.25) (layer Vorderseite) (net 14))
   (segment (start 132.825 99.75) (end 133.55 99.75) (width 0.25) (layer Vorderseite) (net 15) (status 400000))
   (segment (start 135.6 102.1) (end 135.6491 102.09888) (width 0.25) (layer Vorderseite) (net 15) (status C00000))

Commit message: new design
Parts:
- removed C101, C103: 100nF, kicad-libraries:C0603F
- removed C102: 2.2uF, kicad-libraries:C0603F
- removed C104: 10uF, kicad-libraries:C0805
- removed C105: CP1, ELKO_83
- removed Fiducial_Mark (x3): VAL**, kicad-libraries:Fiducial_Mark
- removed G***: Logo_31x31, kicad-libraries:Logo_31x31
- removed G***: LOGO, kicad-libraries:Logo_CoMCU
- removed J101: green, OQ_2P
- removed L101: 10µH, NR4040
- removed R101, R102, R107: 1k, R0603F
- removed R103, R108: 0, R0603F
- removed R104: 390k, R0603F
- removed R105: TBD, R0603F
- removed R106: 10k, R0603F
- removed RP101: 1k, kicad-libraries:4X0603
- removed U101: MCP4551T-104E/MS, MSOP-8
- removed U102: TLV61046A, SOT23-6
- removed VAL: WEEE_7mm, kicad-libraries:WEEE_7mm
- removed VAL: CE_5mm, kicad-libraries:CE_5mm
- added C11: 27nF, kicad-libraries:C0603F, F.Cu at (146.0, 91.0)
- added C12: 2,2nF, kicad-libraries:C0603F, F.Cu at (142.4, 91.8)
- added C13: 120nF, kicad-libraries:C0603F, F.Cu at (143.9, 91.8)
- added C14: 10uF 50V, kicad-libraries:ELKO_63, F.Cu at (152.9, 100.7)
- added C15: 680nF 50V, kicad-libraries:C0603F, F.Cu at (158.1, 103.0)
- added C16: 220uF 50V, kicad-libraries:ELKO_83, F.Cu at (154.0, 108.4)
- added C17: 220uF 50V, kicad-libraries:ELKO_83, F.Cu at (131.0, 114.8)
- added C5: 1uF, kicad-libraries:C0603F, F.Cu at (168.5, 107.7)
- added C7: 10uF, kicad-libraries:C0805E, F.Cu at (147.2, 84.4)
- added C8: 100nF, kicad-libraries:C0603F, F.Cu at (149.2, 84.6)
- added C9: 100nF, kicad-libraries:C0603F, F.Cu at (171.4, 106.4)
- added D3: PMEG4050, kicad-libraries:SOD-128, F.Cu at (153.4, 95.7)
- added L1: SRN8040-100M/10uH, kicad-libraries:SRN8040, F.Cu at (154.6, 89.8)
- added P4: CONN_01X02, kicad-libraries:AKL_5_2_508_green, F.Cu at (142.0, 114.8)
- added Q1: FQD10N20C, kicad-libraries:TO-252-3L, F.Cu at (144.6, 106.4)
- added R1: 1k, kicad-libraries:R0603F, F.Cu at (169.7, 116.9)
- added R10: 1k, kicad-libraries:R0603F, F.Cu at (175.1, 112.4)
- added R13: 220k, kicad-libraries:R0603F, F.Cu at (142.4, 96.1)
- added R14: 10k, kicad-libraries:R0603F, F.Cu at (143.8, 96.1)
- added R3: 470k, kicad-libraries:R0603F, F.Cu at (172.5, 113.6)
- added R4: 68k, kicad-libraries:R0603F, F.Cu at (174.4, 110.8)
- added R7: 60, kicad-libraries:R0603F, F.Cu at (145.9, 96.8)
- added R8: 2k, kicad-libraries:R0603F, F.Cu at (143.2, 94.0)
- added R9: 10k, kicad-libraries:R0603F, F.Cu at (175.5, 102.5)
- added U2: OPA1678, kicad-libraries:SOIC8, F.Cu at (130.9, 104.7)
- added U7: TPS55340, kicad-libraries:S-PWQFN-N16, F.Cu at (147.8, 94.0)
- moved C4 47.1 mm to (177.4, 94.7), turned to 90 degrees
- moved RP1 45.9 mm to (173.8, 95.7), turned to 0 degrees
- moved C1 45.5 mm to (172.4, 102.2), turned to 0 degrees
- moved C2 44.0 mm to (171.2, 95.6), turned to 0 degrees
- moved C3 41.4 mm to (165.3, 109.5), turned to 0 degrees
- moved P3 41.2 mm to (168.2, 101.5)
- moved U4 39.6 mm to (122.5, 117.5)
- moved U5 36.9 mm to (157.5, 117.5)
- moved U6 34.3 mm to (157.5, 82.5)
- moved D1 33.6 mm to (174.3, 107.7), turned to 0 degrees
- moved RP3 32.6 mm to (169.1, 99.5), turned to 0 degrees
- moved P1 21.9 mm to (140.0, 80.0), turned to 180 degrees
- moved D2 20.2 mm to (168.6, 113.6), turned to 90 degrees
- moved U3 18.1 mm to (122.5, 82.5)
- moved U1 12.2 mm to (129.3, 86.3), turned to 270 degrees
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Connections:
- RP3 pad 2: (no net) -> Net-(RP3-Pad2)
- RP3 pad 3: (no net) -> Net-(RP3-Pad3)
- RP3 pad 6: (no net) -> Net-(RP3-Pad6)
- RP3 pad 7: (no net) -> Net-(RP3-Pad7)
- U1 pad 11: (no net) -> Net-(U1-Pad11)
- U1 pad 16: (no net) -> Net-(P3-Pad2)
- U1 pad 17: SDA -> Net-(U1-Pad17)
- U1 pad 18: (no net) -> Net-(U1-Pad18)
- U1 pad 19: SCL -> Net-(U1-Pad19)
- U1 pad 2: EN-PWR -> Enable
- U1 pad 20: (no net) -> Enable
- U1 pad 21: (no net) -> Net-(U1-Pad21)
- U1 pad 3: Net-(P3-Pad2) -> FB0
- U1 pad 4: (no net) -> Net-(U1-Pad4)
- U1 pad 5: (no net) -> Net-(U1-Pad5)
- U1 pad 6: VOUT -> Net-(U1-Pad6)
- U1 pad 7: (no net) -> Net-(U1-Pad7)
- U1 pad 8: (no net) -> Net-(U1-Pad8)
Routing:
- net VCC: track 76.2 -> 0.00 mm, vias 5 -> 0
- net GND: track 47.1 -> 0.00 mm, vias 43 -> 0
- net EN-PWR: track 35.9 -> 0.00 mm, vias 2 -> 0
- net Net-(C104-Pad1): track 31.8 -> 0.00 mm
- net VOUT: track 31.3 -> 0.00 mm, vias 2 -> 0
- net Net-(D2-Pad2): track 25.0 -> 0.00 mm
- net 5V: track 16.7 -> 0.00 mm
- net SCL: track 16.1 -> 0.00 mm, vias 2 -> 0
- net SDA: track 13.3 -> 0.00 mm, vias 2 -> 0
- net POT: track 11.0 -> 0.00 mm
- net Net-(R1-Pad1): track 9.73 -> 0.00 mm, vias 2 -> 0
- net S-CS: track 5.30 -> 0.00 mm
- net S-MISO: track 4.68 -> 0.00 mm
- net S-CLK: track 4.53 -> 0.00 mm
- net Net-(RP3-Pad1): track 4.38 -> 0.00 mm
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- removed copper zone on F.Cu, net 5V
- removed copper zone on B.Cu, net GND
- removed copper zone on F.Cu, net Net-(L101-Pad2)
Other:
- board size 40 x 25 mm -> 40 x 40 mm
- board text removed: "Output"
- board text removed: "PWR"
- board text removed: "Power Supply 1.0"
- board text removed: "Status"
- board text removed: "tinkerforge.com"

Commit message: changes
Parts:
- P4: value CONN_01X02 -> Output; footprint kicad-libraries:AKL_5_2_508_green -> kicad-libraries:OQ_8P
- moved C17 10.3 mm to (126.7, 105.5)
- moved U2 8.77 mm to (126.8, 97.0)
- moved C16 8.50 mm to (146.5, 104.4), turned to 270 degrees
- moved Q1 7.15 mm to (137.4, 106.2), turned to 180 degrees
- moved C15 6.54 mm to (151.7, 104.4), turned to 90 degrees
- moved D3 5.21 mm to (158.1, 98.0), turned to 90 degrees
- moved C14 4.65 mm to (155.7, 104.4), turned to 270 degrees
- moved P4 3.48 mm to (140.0, 112.0)
- moved C8 0.89 mm to (149.6, 85.4)
- moved R13 0.89 mm to (142.8, 96.9)
- moved R14 0.89 mm to (144.2, 96.9)
- moved R7 0.89 mm to (146.3, 97.7)
- moved C11 0.89 mm to (146.4, 91.8)
- moved C12 0.89 mm to (142.8, 92.6)
- moved C13 0.89 mm to (144.3, 92.6)
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Routing:
- added copper zone on F.Cu, net +VSW
- added copper zone on F.Cu, net 5V
- added copper zone on F.Cu, net GND
- added copper zone on F.Cu, net Net-(D3-Pad1)
- added copper zone on F.Cu, net Vo0

Commit message: changes
Parts:
- added C6: 10uF, kicad-libraries:C0805E, F.Cu at (145.8, 87.8)
- moved Q1 4.79 mm to (139.1, 101.7), turned to 270 degrees
- moved D3 4.34 mm to (154.1, 96.4), turned to 180 degrees
- moved C7 2.60 mm to (147.8, 87.8), turned to 270 degrees
- moved C8 2.41 mm to (149.3, 87.8), turned to 270 degrees
- moved C14 1.99 mm to (156.3, 102.5), turned to 90 degrees
- moved C15 1.92 mm to (152.2, 102.5), turned to 270 degrees
- moved C17 0.67 mm to (126.4, 106.0)
- moved C16 0.49 mm to (146.9, 104.2), turned to 90 degrees

Commit message: changes
Parts:
- removed RP3: 1k, kicad-libraries:4X0603
- added R2: 1k, kicad-libraries:R0603F, F.Cu at (130.1, 82.5)
- added R5: 1k, kicad-libraries:R0603F, F.Cu at (148.5, 82.5)
- D2: value green -> red
- moved R10 51.5 mm to (124.9, 100.8), turned to 180 degrees
- moved C4 51.1 mm to (126.5, 88.8)
- moved D1 49.7 mm to (131.5, 82.5), turned to 90 degrees
- moved P3 47.7 mm to (122.5, 88.0)
- moved R9 47.5 mm to (128.0, 100.8), turned to 180 degrees
- moved R1 46.9 mm to (129.2, 93.2), turned to 270 degrees
- moved R4 46.2 mm to (130.7, 96.2), turned to 270 degrees
- moved R3 44.0 mm to (132.1, 96.2)
- moved C9 43.4 mm to (129.2, 96.2), turned to 270 degrees
- moved C1 41.3 mm to (134.7, 85.5), turned to 180 degrees
- moved RP1 40.1 mm to (134.7, 87.1), turned to 90 degrees
- moved C5 39.5 mm to (131.4, 94.0)
- moved D2 36.1 mm to (150.1, 82.5)
- moved C3 31.7 mm to (141.9, 88.0)
- moved C2 30.6 mm to (141.9, 86.5)
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Connections:
- U1 pad 12: Net-(R1-Pad1) -> Net-(R2-Pad1)
- U1 pad 13: Net-(RP3-Pad1) -> Net-(R1-Pad1)
- U1 pad 15: Net-(P2-Pad1) -> Net-(U1-Pad15)
- U1 pad 16: Net-(P3-Pad2) -> Net-(U1-Pad16)
- U1 pad 2: Enable -> Net-(U1-Pad2)
- U1 pad 7: Net-(U1-Pad7) -> Net-(P2-Pad1)
- U1 pad 8: Net-(U1-Pad8) -> Net-(P3-Pad2)
- U2 pad 1: Net-(U2-Pad1) -> Net-(Q1-PadG)
- U2 pad 2: Net-(U2-Pad2) -> Net-(C9-Pad1)
- U2 pad 3: Net-(U2-Pad3) -> PWM0
- U2 pad 5: PWM0 -> Net-(U2-Pad5)
- U2 pad 6: Net-(C9-Pad1) -> Net-(U2-Pad6)
- U2 pad 7: Net-(Q1-PadG) -> Net-(U2-Pad7)
Routing:
- net VCC: track 0.00 -> 40.2 mm, vias 0 -> 4
- net Net-(R5-Pad1): track 0.00 -> 34.4 mm, vias 0 -> 2
- net FB0: track 0.00 -> 29.7 mm
- net +VSW: track 0.00 -> 20.6 mm
- net Enable: track 0.00 -> 18.2 mm
- net Net-(R2-Pad1): track 0.00 -> 16.7 mm, vias 0 -> 2
- net GND: track 0.00 -> 15.8 mm, vias 0 -> 115
- net Vo0: track 0.00 -> 10.4 mm, vias 0 -> 2
- net 5V: track 0.00 -> 9.83 mm
- net Net-(P3-Pad2): track 0.00 -> 8.20 mm
- net Net-(P2-Pad1): track 0.00 -> 7.14 mm
- net Net-(Q1-PadG): track 0.00 -> 6.75 mm
- net Net-(P1-Pad4): track 0.00 -> 6.72 mm
- net Net-(P1-Pad5): track 0.00 -> 5.26 mm
- net Net-(C9-Pad1): track 0.00 -> 4.50 mm
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- added copper zone on B.Cu, net GND
- added copper zone on F.Cu, net VCC
Other:
- net class Default: clearance 0.15 -> 0.149
- rule trace_clearance: 0.15 -> 0.149
- board text added: "Failure"

Commit message: final prototype design
Parts:
- added Fiducial_Mark: VAL**, kicad-libraries:Fiducial_Mark, F.Cu at (157.0, 109.0)
- added Fiducial_Mark: VAL**, kicad-libraries:Fiducial_Mark, F.Cu at (153.0, 83.0)
- added Fiducial_Mark: VAL**, kicad-libraries:Fiducial_Mark, F.Cu at (122.0, 100.0)
- added G***: LOGO, kicad-libraries:Logo_31x31, F.Cu at (137.5, 95.2)
- added G***: LOGO, kicad-libraries:Logo_CoMCU, B.Cu at (146.5, 100.0)
- added VAL: WEEE_7mm, kicad-libraries:WEEE_7mm, B.Cu at (140.0, 100.0)
- added VAL: CE_5mm, kicad-libraries:CE_5mm, B.Cu at (134.0, 100.0)
- D2: value red -> green
Other:
- board text added: "+"
- board text added: "-"
- board text added: "Industrial Power Supply 1.0"
- board text added: "Output"
- board text added: "Status"
- board text added: "VOut"
- board text added: "max. ??W"
- board text added: "tinkerforge.com"
- board text removed: "Failure"
